Commit message: update jazzy
Signed-off-by: Stevedan Omodolor <stevedan.o.omodolor@gmail.com>

File: nav2_minimal_tb3_sim/urdf/gz_waffle_gps.sdf.xacro (robot description, xacro)
@@ -98,4 +98,6 @@
             <position_sensing>
               <horizontal>
+              <!-- Be carefull setting this.
+              Units in degree not in meters https://github.com/gazebosim/sdformat/issues/1572 -->
                 <noise type="gaussian">
                   <mean>0.0</mean>
@@ -144,5 +146,5 @@
           </geometry>
           <material>
-            <diffuse>1 1 1</diffuse>
+            <diffuse>0.5 0.5 0.5</diffuse>
           </material>
         </visual>
@@ -199,5 +201,5 @@
           <surface>
             <friction>
-              <ode>
+              <bullet>
                 <mu>1</mu>
                 <mu2>1</mu2>
@@ -205,8 +207,8 @@
                 <slip2>0</slip2>
                 <fdir1>0 0 1</fdir1>
-              </ode>
+              </bullet>
             </friction>
             <contact>
-              <ode>
+              <bullet>
                 <soft_cfm>0</soft_cfm>
                 <soft_erp>0.2</soft_erp>
@@ -215,5 +217,5 @@
                 <max_vel>0.01</max_vel>
                 <min_depth>0.001</min_depth>
-              </ode>
+              </bullet>
             </contact>
           </surface>
@@ -228,5 +230,5 @@
           </geometry>
           <material>
-            <diffuse>1 1 1</diffuse>
+            <diffuse>0.5 0.5 0.5</diffuse>
           </material>
         </visual>
@@ -255,5 +257,5 @@
           <surface>
             <friction>
-              <ode>
+              <bullet>
                 <mu>1</mu>
                 <mu2>1</mu2>
@@ -261,8 +263,8 @@
                 <slip2>0</slip2>
                 <fdir1>0 0 1</fdir1>
-              </ode>
+              </bullet>
             </friction>
             <contact>
-              <ode>
+              <bullet>
                 <soft_cfm>0</soft_cfm>
                 <soft_erp>0.2</soft_erp>
@@ -271,5 +273,5 @@
                 <max_vel>0.01</max_vel>
                 <min_depth>0.001</min_depth>
-              </ode>
+              </bullet>
             </contact>
           </surface>
@@ -284,10 +286,10 @@
           </geometry>
           <material>
-            <diffuse>1 1 1</diffuse>
+            <diffuse>0.5 0.5 0.5</diffuse>
           </material>
         </visual>
       </link>
       <link name='caster_back_right_link'>
-        <pose>-0.177 -0.064 -0.004 0 0 0</pose>
+        <pose>-0.177 -0.064 -0.004 -1.57 0 0</pose>
         <inertial>
           <mass>0.001</mass>
@@ -304,10 +306,10 @@
           <geometry>
             <sphere>
-              <radius>0.005000</radius>
+              <radius>0.006000</radius>
             </sphere>
           </geometry>
           <surface>
             <contact>
-              <ode>
+              <bullet>
                 <soft_cfm>0</soft_cfm>
                 <soft_erp>0.2</soft_erp>
@@ -316,11 +318,21 @@
                 <max_vel>0.01</max_vel>
                 <min_depth>0.001</min_depth>
-              </ode>
+              </bullet>
             </contact>
           </surface>
         </collision>
+        <visual name="sphere_visual">
+          <geometry>
+            <sphere>
+              <radius>0.0060000</radius>
+            </sphere>
+          </geometry>
+          <material>
+            <diffuse>0.5 0.5 0.5</diffuse>
+          </material>
+        </visual>
       </link>
       <link name='caster_back_left_link'>
-        <pose>-0.177 0.064 -0.004 0 0 0</pose>
+        <pose>-0.177 0.064 -0.004 -1.57 0 0</pose>
         <inertial>
           <mass>0.001</mass>
@@ -337,10 +349,10 @@
           <geometry>
             <sphere>
-              <radius>0.005000</radius>
+              <radius>0.006000</radius>
             </sphere>
           </geometry>
           <surface>
             <contact>
-              <ode>
+              <bullet>
                 <soft_cfm>0</soft_cfm>
                 <soft_erp>0.2</soft_erp>
@@ -349,8 +361,18 @@
                 <max_vel>0.01</max_vel>
                 <min_depth>0.001</min_depth>
-              </ode>
+              </bullet>
             </contact>
           </surface>
         </collision>
+        <visual name="sphere_visual">
+          <geometry>
+            <sphere>
+              <radius>0.0060000</radius>
+            </sphere>
+          </geometry>
+          <material>
+            <diffuse>0.5 0.5 0.5</diffuse>
+          </material>
+        </visual>
       </link>
       <link name="camera_link">
